File: kicad/genesis_6button/genesis_6button.kicad_pcb (KiCad board)
At the start: 2 copper layers, 73.7 x 36.8 mm, 21 parts, among them J1 Conn_02x07_Odd_Even, J2 DB9_Female, J3 Conn_02x03_Odd_Even, U1 74LS257, U2 ATtiny204-SS, U3 74LS257

Commit message: Change to actual component values + comments
Parts:
- U1, U3: value 74LS257 -> 74HC257
- U2: value ATtiny204-SS -> ATtiny404-SS
Changed lines of the file:
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@@
       (effects (font (size 1 1) (thickness 0.15)))
     )
-    (fp_text value 74LS257 (at 0 5.9) (layer F.Fab)
+    (fp_text value 74HC257 (at 0 5.9) (layer F.Fab)
       (effects (font (size 1 1) (thickness 0.15)))
     )
@@
       (effects (font (size 1 1) (thickness 0.15)))
     )
-    (fp_text value ATtiny204-SS (at 0 5.28 90) (layer F.Fab)
+    (fp_text value ATtiny404-SS (at 0 5.28 90) (layer F.Fab)
       (effects (font (size 1 1) (thickness 0.15)))
     )
@@
       (effects (font (size 1 1) (thickness 0.15)))
     )
-    (fp_text value 74LS257 (at 0 5.9) (layer F.Fab)
+    (fp_text value 74HC257 (at 0 5.9) (layer F.Fab)
       (effects (font (size 1 1) (thickness 0.15)))
     )

Commit message: Second PCB iteration (untested)
Parts:
- added C4: 10u, Capacitor_THT:CP_Radial_D8.0mm_P5.00mm, F.Cu at (134.9, 43.0)
- added R13: 100k, Resistor_SMD:R_0805_2012Metric, F.Cu at (141.7, 55.4)
- added R14: 100k, Resistor_SMD:R_0805_2012Metric, F.Cu at (146.7, 55.4)
- added TP1: TestPoint, TestPoint:TestPoint_Loop_D3.50mm_Drill0.9mm_Beaded, F.Cu at (115.0, 41.6)
- added TP2: TestPoint, TestPoint:TestPoint_Loop_D3.50mm_Drill0.9mm_Beaded, F.Cu at (107.6, 41.6)
- C1, C2, C3: footprint Capacitor_SMD:C_0805_2012Metric -> Capacitor_SMD:C_1206_3216Metric
- R1, R10, R11, R12, R2, R3, R4, R5, R6, R7, R8, R9: value 47k -> 75k
- moved C2 0.20 mm to (139.5, 49.8)
- moved C3 0.15 mm to (129.1, 59.8)
Connections:
- U2 pad 3: (no net) -> BUTTON_MODE
- U3 pad 2: BUTTON_UP -> BUTTON_DOWN
- U3 pad 3: BUTTON_Z -> BUTTON_Y
- U3 pad 4: UP -> DOWN
- U3 pad 5: BUTTON_DOWN -> BUTTON_UP
- U3 pad 6: BUTTON_Y -> BUTTON_Z
- U3 pad 7: DOWN -> UP
Routing:
- net Net-(J3-Pad1): track 77.9 -> 30.3 mm, vias 2 -> 1
- net BUTTON_Z: track 74.1 -> 59.7 mm, vias 2 -> 0
- net +5V: track 168.2 -> 154.6 mm, vias 5 -> 2
- net BUTTON_MODE: track 61.3 -> 74.5 mm, vias 4 -> 5
- net BUTTON_Y: track 64.9 -> 53.4 mm, vias 2 -> 0
- net DOWN: track 81.8 -> 70.5 mm
- net BUTTON_UP: track 29.0 -> 40.0 mm
- net BUTTON_X: track 71.4 -> 60.6 mm
- net TH: track 75.8 -> 69.0 mm
- net Net-(R14-Pad2): track 28.9 -> 35.1 mm
- net BUTTON_C: track 30.4 -> 35.6 mm
- net BUTTON_DOWN: track 34.1 -> 29.3 mm, vias 2 -> 1
- net UP: track 76.4 -> 73.3 mm
- net BUTTON_START: track 41.4 -> 44.4 mm
- net TR: track 53.4 -> 50.5 mm
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Other:
- board size 73.7 x 36.8 mm -> 70.4 x 36.8 mm
- board text added: "+5V"
- board text added: "GND"

Commit message: Add hole for cable tie + replace/route
Parts:
- added H1: MountingHole, MountingHole:MountingHole_5.3mm_M5, F.Cu at (157.1, 43.5)
- moved J2 4.96 mm to (153.9, 50.7)
Routing:
- net DOWN: track 70.5 -> 55.3 mm, vias 1 -> 4
- net +5V: track 154.6 -> 139.7 mm, vias 2 -> 3
- net RIGHT: track 44.0 -> 52.7 mm, vias 2 -> 3
- net UP: track 73.3 -> 66.3 mm, vias 1 -> 2
- net Net-(R14-Pad2): track 35.1 -> 41.7 mm
- net LEFT: track 41.5 -> 47.4 mm
- net TR: track 50.5 -> 54.8 mm
- net TH: track 69.0 -> 72.9 mm
- net TL: track 40.1 -> 38.8 mm
- net GND: vias 26 -> 24

Commit message: Shrink board.
Parts:
- moved TP2 33.4 mm to (120.2, 72.5)
- moved R4 16.5 mm to (119.4, 64.7), turned to 270 degrees
- moved R5 15.8 mm to (114.5, 64.7), turned to 270 degrees
- moved R11 14.4 mm to (119.4, 51.8), turned to 270 degrees
- moved R6 12.2 mm to (114.5, 58.1), turned to 270 degrees
- moved R12 11.4 mm to (119.4, 58.1), turned to 270 degrees
- moved R10 9.76 mm to (116.9, 51.8), turned to 270 degrees
- moved R7 9.15 mm to (116.9, 64.7), turned to 270 degrees
- moved R1 8.10 mm to (116.9, 46.1), turned to 270 degrees
- moved J1 8.05 mm to (105.1, 49.3)
- moved R3 7.22 mm to (119.4, 46.1), turned to 270 degrees
- moved R8 6.67 mm to (116.9, 58.1), turned to 270 degrees
- moved R9 6.43 mm to (114.5, 51.8), turned to 270 degrees
- moved TP1 5.56 mm to (120.4, 40.4)
- moved R2 4.65 mm to (114.5, 46.1), turned to 270 degrees
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Routing:
- net BUTTON_Y: track 53.4 -> 29.6 mm, vias 0 -> 1
- net BUTTON_Z: track 59.7 -> 35.9 mm, vias 0 -> 2
- net BUTTON_X: track 60.6 -> 39.0 mm, vias 2 -> 3
- net BUTTON_LEFT: track 66.6 -> 48.5 mm, vias 3 -> 2
- net BUTTON_UP: track 40.0 -> 22.7 mm
- net BUTTON_MODE: track 74.5 -> 59.7 mm, vias 5 -> 3
- net BUTTON_C: track 35.6 -> 21.0 mm, vias 1 -> 0
- net BUTTON_A: track 33.6 -> 25.9 mm, vias 1 -> 2
- net BUTTON_B: track 30.1 -> 22.6 mm, vias 1 -> 0
- net BUTTON_DOWN: track 29.3 -> 25.0 mm, vias 1 -> 2
- net DOWN: track 55.3 -> 52.2 mm
- net Net-(R13-Pad2): track 26.4 -> 28.5 mm
- net TH: track 72.9 -> 74.3 mm
- net BUTTON_START: track 44.4 -> 43.0 mm, vias 2 -> 3
- net TR: track 54.8 -> 53.6 mm
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Other:
- board size 70.4 x 36.8 mm -> 61.7 x 36.8 mm
